Commit message: simulation works now

File: assets/excavator_4dof/excavator_4dof.urdf (robot description, URDF)
Before this commit: robot excavator_4dof, 6 links, 5 joints
Links:
- removed link world
- link arm_link: geometry visual box size=1.6 0.28 0.28
- link boom_link: geometry visual box size=2.0 0.35 0.35
- link bucket_link: mass 350.0 -> 220.0; geometry collision box size=0.02 0.5 0.4; collision box size=0.6 0.02 0.4
- link house_link: geometry visual box size=1.4 1.2 0.9
Joints:
- removed joint world_fixed
- joint arm_joint: limit lower=-1.4 upper=0.6 effort=5000 velocity=0.9 -> lower=-1.57 upper=1.57 effort=5000 velocity=0.9; origin xyz=2.0 0 0 rpy=0 0 0 -> xyz=2.0 0 0 rpy=0 1.57 0
- joint boom_joint: limit lower=-0.3 upper=1.2 effort=7000 velocity=0.7 -> lower=-0.79 upper=0.79 effort=7000 velocity=0.7; origin xyz=0.65 0 0.75 rpy=0 0 0 -> xyz=0.65 0 0.75 rpy=0 -0.79 0
- joint bucket_joint: limit lower=-1.8 upper=0.8 effort=3500 velocity=1.2 -> lower=-1.57 upper=1.57 effort=3500 velocity=1.2; origin xyz=1.6 0 0 rpy=0 0 0 -> xyz=1.6 0 -0.15 rpy=0 -1.57 0

Commit message: add two cameras and debugging lidar

File: assets/excavator_4dof/excavator_4dof.urdf (robot description, URDF)
Before this commit: robot excavator_4dof, 5 links, 4 joints
Joints:
- joint boom_joint: origin xyz=0.65 0 0.75 rpy=0 -0.79 0 -> xyz=0.7 -0.4 0.9 rpy=0 -0.79 0
- joint bucket_joint: origin xyz=1.6 0 -0.15 rpy=0 -1.57 0 -> xyz=1.6 0 0.0 rpy=0 -1.57 0
